Commit message: add joint limits to match bastian robotics

File: fanuc_m10id_support/urdf/m10id12_macro.xacro (robot description, xacro)
@@ -144,5 +144,5 @@
       <child link="${prefix}link_5"/>
       <axis xyz="0 -1 0"/>
-      <limit lower="-3.14" upper="3.14" effort="0" velocity="7.85"/>
+      <limit lower="-2.443" upper="2.443" effort="0" velocity="7.85"/>
     </joint>
     <joint name="${prefix}joint_6" type="revolute">
@@ -151,5 +151,5 @@
       <child link="${prefix}link_6"/>
       <axis xyz="-1 0 0"/>
-      <limit lower="-7.85" upper="7.85" effort="0" velocity="12.56"/>
+      <limit lower="-4.71239" upper="4.71239" effort="0" velocity="12.56"/>
     </joint>
     <!-- ROS-Industrial 'base' frame: base_link to Fanuc World Coordinates transform -->

Commit message: reduce even more for geoff

File: fanuc_m10id_support/urdf/m10id12_macro.xacro (robot description, xacro)
@@ -151,5 +151,5 @@
       <child link="${prefix}link_6"/>
       <axis xyz="-1 0 0"/>
-      <limit lower="-4.71239" upper="4.71239" effort="0" velocity="12.56"/>
+      <limit lower="-3.22886" upper="3.22886" effort="0" velocity="12.56"/>
     </joint>
     <!-- ROS-Industrial 'base' frame: base_link to Fanuc World Coordinates transform -->

Commit message: fixed numbers to match

File: fanuc_m10id_support/urdf/m10id12_macro.xacro (robot description, xacro)
@@ -106,4 +106,80 @@
         <geometry>
           <mesh filename="package://fanuc_m10id_support/meshes/m10id12/collision/link_6.stl"/>
+        </geometry>
+      </collision>
+    </link>
+<!-- DCS ZONE LINKS: 5 zone links starting at link_2 -->
+    <link name="dcs_z2">
+      <visual>
+        <origin xyz="0 0 0" rpy="0 0 0"/>
+        <geometry>
+          <mesh filename="package://fanuc_m10id_support/meshes/m10id12/visual/dcs_z2.stl"/>
+        </geometry>
+        <!-- <xacro:material_fanuc_black /> -->
+      </visual>
+      <collision>
+        <origin xyz="0 0 0" rpy="0 0 0"/>
+        <geometry>
+          <mesh filename="package://fanuc_m10id_support/meshes/m10id12/collision/dcs_z2.stl"/>
+        </geometry>
+      </collision>
+    </link>
+    <link name="dcs_z3">
+      <visual>
+        <origin xyz="0 0 0" rpy="0 0 0"/>
+        <geometry>
+          <mesh filename="package://fanuc_m10id_support/meshes/m10id12/visual/dcs_z3.stl"/>
+        </geometry>
+        <!-- <xacro:material_fanuc_black /> -->
+      </visual>
+      <collision>
+        <origin xyz="0 0 0" rpy="0 0 0"/>
+        <geometry>
+          <mesh filename="package://fanuc_m10id_support/meshes/m10id12/collision/dcs_z3.stl"/>
+        </geometry>
+      </collision>
+    </link>
+    <link name="dcs_z4">
+      <visual>
+        <origin xyz="0 0 0" rpy="0 0 0"/>
+        <geometry>
+          <mesh filename="package://fanuc_m10id_support/meshes/m10id12/visual/dcs_z4.stl"/>
+        </geometry>
+        <!-- <xacro:material_fanuc_black /> -->
+      </visual>
+      <collision>
+        <origin xyz="0 0 0" rpy="0 0 0"/>
+        <geometry>
+          <mesh filename="package://fanuc_m10id_support/meshes/m10id12/collision/dcs_z4.stl"/>
+        </geometry>
+      </collision>
+    </link>
+    <link name="dcs_z5">
+      <visual>
+        <origin xyz="0 0 0" rpy="0 0 0"/>
+        <geometry>
+          <mesh filename="package://fanuc_m10id_support/meshes/m10id12/visual/dcs_z5.stl"/>
+        </geometry>
+        <!-- <xacro:material_fanuc_black /> -->
+      </visual>
+      <collision>
+        <origin xyz="0 0 0" rpy="0 0 0"/>
+        <geometry>
+          <mesh filename="package://fanuc_m10id_support/meshes/m10id12/collision/dcs_z5.stl"/>
+        </geometry>
+      </collision>
+    </link>
+    <link name="dcs_z6">
+      <visual>
+        <origin xyz="0 0 0" rpy="0 0 0"/>
+        <geometry>
+          <mesh filename="package://fanuc_m10id_support/meshes/m10id12/visual/dcs_z6.stl"/>
+        </geometry>
+        <!-- <xacro:material_fanuc_black /> -->
+      </visual>
+      <collision>
+        <origin xyz="0 0 0" rpy="0 0 0"/>
+        <geometry>
+          <mesh filename="package://fanuc_m10id_support/meshes/m10id12/collision/dcs_z6.stl"/>
         </geometry>
       </collision>
@@ -174,4 +250,30 @@
       <child link="${prefix}tool0" />
     </joint>
+<!-- DCS JOINTS -->
+    <joint name="dcs_z1-joint" type="fixed">
+      <origin xyz="-0.175 0 0.127" rpy="0 0 0"/>
+      <parent link="${prefix}link_1"/>
+      <child link="dcs_z1"/>
+    </joint>
+    <joint name="dcs_z2-joint" type="fixed">
+      <origin xyz="-0.035 -0.04 0.02" rpy="0 0 0"/>
+      <parent link="${prefix}link_2"/>
+      <child link="dcs_z2"/>
+    </joint>
+    <joint name="dcs_z3-joint" type="fixed">
+      <origin xyz="0.085 0.01 -0.14" rpy="0 0 0"/>
+      <parent link="${prefix}link_3"/>
+      <child link="dcs_z3"/>
+    </joint>
+    <joint name="dcs_z4-joint" type="fixed">
+      <origin xyz="0.041 0.07 0" rpy="0 0 0"/>
+      <parent link="${prefix}link_4"/>
+      <child link="dcs_z4"/>
+    </joint>
+    <joint name="dcs_z5-joint" type="fixed">
+      <origin xyz="0.035 0.057 -0.065" rpy="0 0 0"/>
+      <parent link="${prefix}link_5"/>
+      <child link="dcs_z5"/>
+    </joint>
   </xacro:macro>
 </robot>

Commit message: now the numbers are fixed

File: fanuc_m10id_support/urdf/m10id12_macro.xacro (robot description, xacro)
@@ -110,16 +110,31 @@
     </link>
 <!-- DCS ZONE LINKS: 5 zone links starting at link_2 -->
+    <link name="dcs_z1">
+      <visual>
+        <origin xyz="0 0 0" rpy="0 0 0"/>
+        <geometry>
+          <mesh filename="package://fanuc_m10id_support/meshes/m10id12/visual/dcs_z2.stl"/>
+        </geometry>
+        <!-- <xacro:material_fanuc_black /> -->
+      </visual>
+      <collision>
+        <origin xyz="0 0 0" rpy="0 0 0"/>
+        <geometry>
+          <mesh filename="package://fanuc_m10id_support/meshes/m10id12/collision/dcs_z2.stl"/>
+        </geometry>
+      </collision>
+    </link>
     <link name="dcs_z2">
       <visual>
         <origin xyz="0 0 0" rpy="0 0 0"/>
         <geometry>
-          <mesh filename="package://fanuc_m10id_support/meshes/m10id12/visual/dcs_z2.stl"/>
-        </geometry>
-        <!-- <xacro:material_fanuc_black /> -->
-      </visual>
-      <collision>
-        <origin xyz="0 0 0" rpy="0 0 0"/>
-        <geometry>
-          <mesh filename="package://fanuc_m10id_support/meshes/m10id12/collision/dcs_z2.stl"/>
+          <mesh filename="package://fanuc_m10id_support/meshes/m10id12/visual/dcs_z3.stl"/>
+        </geometry>
+        <!-- <xacro:material_fanuc_black /> -->
+      </visual>
+      <collision>
+        <origin xyz="0 0 0" rpy="0 0 0"/>
+        <geometry>
+          <mesh filename="package://fanuc_m10id_support/meshes/m10id12/collision/dcs_z3.stl"/>
         </geometry>
       </collision>
@@ -129,12 +144,12 @@
         <origin xyz="0 0 0" rpy="0 0 0"/>
         <geometry>
-          <mesh filename="package://fanuc_m10id_support/meshes/m10id12/visual/dcs_z3.stl"/>
-        </geometry>
-        <!-- <xacro:material_fanuc_black /> -->
-      </visual>
-      <collision>
-        <origin xyz="0 0 0" rpy="0 0 0"/>
-        <geometry>
-          <mesh filename="package://fanuc_m10id_support/meshes/m10id12/collision/dcs_z3.stl"/>
+          <mesh filename="package://fanuc_m10id_support/meshes/m10id12/visual/dcs_z4.stl"/>
+        </geometry>
+        <!-- <xacro:material_fanuc_black /> -->
+      </visual>
+      <collision>
+        <origin xyz="0 0 0" rpy="0 0 0"/>
+        <geometry>
+          <mesh filename="package://fanuc_m10id_support/meshes/m10id12/collision/dcs_z4.stl"/>
         </geometry>
       </collision>
@@ -144,31 +159,16 @@
         <origin xyz="0 0 0" rpy="0 0 0"/>
         <geometry>
-          <mesh filename="package://fanuc_m10id_support/meshes/m10id12/visual/dcs_z4.stl"/>
-        </geometry>
-        <!-- <xacro:material_fanuc_black /> -->
-      </visual>
-      <collision>
-        <origin xyz="0 0 0" rpy="0 0 0"/>
-        <geometry>
-          <mesh filename="package://fanuc_m10id_support/meshes/m10id12/collision/dcs_z4.stl"/>
+          <mesh filename="package://fanuc_m10id_support/meshes/m10id12/visual/dcs_z5.stl"/>
+        </geometry>
+        <!-- <xacro:material_fanuc_black /> -->
+      </visual>
+      <collision>
+        <origin xyz="0 0 0" rpy="0 0 0"/>
+        <geometry>
+          <mesh filename="package://fanuc_m10id_support/meshes/m10id12/collision/dcs_z5.stl"/>
         </geometry>
       </collision>
     </link>
     <link name="dcs_z5">
-      <visual>
-        <origin xyz="0 0 0" rpy="0 0 0"/>
-        <geometry>
-          <mesh filename="package://fanuc_m10id_support/meshes/m10id12/visual/dcs_z5.stl"/>
-        </geometry>
-        <!-- <xacro:material_fanuc_black /> -->
-      </visual>
-      <collision>
-        <origin xyz="0 0 0" rpy="0 0 0"/>
-        <geometry>
-          <mesh filename="package://fanuc_m10id_support/meshes/m10id12/collision/dcs_z5.stl"/>
-        </geometry>
-      </collision>
-    </link>
-    <link name="dcs_z6">
       <visual>
         <origin xyz="0 0 0" rpy="0 0 0"/>

Commit message: nope now they are fixed

File: fanuc_m10id_support/urdf/m10id12_macro.xacro (robot description, xacro)
@@ -114,4 +114,19 @@
         <origin xyz="0 0 0" rpy="0 0 0"/>
         <geometry>
+          <mesh filename="package://fanuc_m10id_support/meshes/m10id12/visual/dcs_z1.stl"/>
+        </geometry>
+        <!-- <xacro:material_fanuc_black /> -->
+      </visual>
+      <collision>
+        <origin xyz="0 0 0" rpy="0 0 0"/>
+        <geometry>
+          <mesh filename="package://fanuc_m10id_support/meshes/m10id12/collision/dcs_z1.stl"/>
+        </geometry>
+      </collision>
+    </link>
+    <link name="dcs_z2">
+      <visual>
+        <origin xyz="0 0 0" rpy="0 0 0"/>
+        <geometry>
           <mesh filename="package://fanuc_m10id_support/meshes/m10id12/visual/dcs_z2.stl"/>
         </geometry>
@@ -125,5 +140,5 @@
       </collision>
     </link>
-    <link name="dcs_z2">
+    <link name="dcs_z3">
       <visual>
         <origin xyz="0 0 0" rpy="0 0 0"/>
@@ -140,5 +155,5 @@
       </collision>
     </link>
-    <link name="dcs_z3">
+    <link name="dcs_z4">
       <visual>
         <origin xyz="0 0 0" rpy="0 0 0"/>
@@ -155,5 +170,5 @@
       </collision>
     </link>
-    <link name="dcs_z4">
+    <link name="dcs_z5">
       <visual>
         <origin xyz="0 0 0" rpy="0 0 0"/>
@@ -167,19 +182,4 @@
         <geometry>
           <mesh filename="package://fanuc_m10id_support/meshes/m10id12/collision/dcs_z5.stl"/>
-        </geometry>
-      </collision>
-    </link>
-    <link name="dcs_z5">
-      <visual>
-        <origin xyz="0 0 0" rpy="0 0 0"/>
-        <geometry>
-          <mesh filename="package://fanuc_m10id_support/meshes/m10id12/visual/dcs_z6.stl"/>
-        </geometry>
-        <!-- <xacro:material_fanuc_black /> -->
-      </visual>
-      <collision>
-        <origin xyz="0 0 0" rpy="0 0 0"/>
-        <geometry>
-          <mesh filename="package://fanuc_m10id_support/meshes/m10id12/collision/dcs_z6.stl"/>
         </geometry>
       </collision>
