Commit message: forgot to push this change which allows the user to toggle a boolean in the cat_universal_robot_cell_urdf_xacro in case they want to debug with a non-capsule robot model and instead use the actual manufacturers stl meshes for robot model

File: fanuc_m10id_support/urdf/m10id12_capsule_macro.xacro (robot description, xacro)
@@ -2,5 +2,5 @@
 <robot xmlns:xacro="http://wiki.ros.org/xacro">
   <xacro:include filename="$(find fanuc_resources)/urdf/common_materials.xacro"/>
-  <xacro:macro name="fanuc_m10id12" params="prefix">
+  <xacro:macro name="fanuc_m10id12_capsule" params="prefix">
     <!-- links: main serial chain -->
     <link name="${prefix}base_link">
